File: 42-stepper-motor-driver-tryout.kicad_sch (KiCad schematic)
At the start: 4 parts

Commit message: update,
Other:
- added sheet MCU (MCU.kicad_sch)
- added sheet drive (drive.kicad_sch)
- added sheet interface (interface.kicad_sch)
- added sheet port (port.kicad_sch)
- added sheet power (power.kicad_sch)
Changed lines of the file:
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@@
+    )
+  )
+  (sheet (at 38.1 63.5) (size 25.4 25.4) (fields_autoplaced)
+    (stroke (width 0.1524) (type solid) (color 0 0 0 0))
+    (fill (color 0 0 0 0.0000))
+    (property "Sheet name" "drive" (id 0) (at 38.1 62.7884 0)
+      (effects (font (size 1.27 1.27)) (justify left bottom))
+    )
+    (property "Sheet file" "drive.kicad_sch" (id 1) (at 38.1 89.4846 0)
+      (effects (font (size 1.27 1.27)) (justify left top))
+    )
+  )
+  (sheet (at 114.3 63.5) (size 25.4 25.4) (fields_autoplaced)
+    (stroke (width 0.1524) (type solid) (color 0 0 0 0))
+    (fill (color 0 0 0 0.0000))
+    (property "Sheet name" "port" (id 0) (at 114.3 62.7884 0)
+      (effects (font (size 1.27 1.27)) (justify left bottom))
+    )
+    (property "Sheet file" "port.kicad_sch" (id 1) (at 114.3 89.4846 0)
+      (effects (font (size 1.27 1.27)) (justify left top))
+    )
+  )
+  (sheet (at 190.5 63.5) (size 25.4 25.4) (fields_autoplaced)
+    (stroke (width 0.1524) (type solid) (color 0 0 0 0))
+    (fill (color 0 0 0 0.0000))
+    (property "Sheet name" "interface" (id 0) (at 190.5 62.7884 0)
+      (effects (font (size 1.27 1.27)) (justify left bottom))
+    )
+    (property "Sheet file" "interface.kicad_sch" (id 1) (at 190.5 89.4846 0)
+      (effects (font (size 1.27 1.27)) (justify left top))
+    )
+  )
+  (sheet (at 76.2 63.5) (size 25.4 25.4) (fields_autoplaced)
+    (stroke (width 0.1524) (type solid) (color 0 0 0 0))
+    (fill (color 0 0 0 0.0000))
+    (property "Sheet name" "MCU" (id 0) (at 76.2 62.7884 0)
+      (effects (font (size 1.27 1.27)) (justify left bottom))
+    )
+    (property "Sheet file" "MCU.kicad_sch" (id 1) (at 76.2 89.4846 0)
+      (effects (font (size 1.27 1.27)) (justify left top))
+    )
+  )
+  (sheet (at 152.4 63.5) (size 25.4 25.4) (fields_autoplaced)
+    (stroke (width 0.1524) (type solid) (color 0 0 0 0))
+    (fill (color 0 0 0 0.0000))
+    (property "Sheet name" "power" (id 0) (at 152.4 62.7884 0)
+      (effects (font (size 1.27 1.27)) (justify left bottom))
+    )
+    (property "Sheet file" "power.kicad_sch" (id 1) (at 152.4 89.4846 0)
+      (effects (font (size 1.27 1.27)) (justify left top))
     )
   )
   (sheet_instances
     (path "/" (page "1"))
+    (path "/17e68860-358f-4811-82c9-1048556048f8" (page "2"))
+    (path "/b63773fb-e66c-408a-b6e1-6a1e3b3ffea6" (page "3"))
+    (path "/4bcdaace-7736-4d61-ba21-98bab1967e94" (page "4"))
+    (path "/d7dee512-1141-4256-b411-29ff8008ec9a" (page "5"))
+    (path "/876e9f45-76fc-4061-9985-ee1c7ce34684" (page "6"))
   )
   (symbol_instances

Commit message: update,
Other:
- moved on the sheet: H1, H2, H3, H4
