File: port.kicad_sch (KiCad schematic)
At the start: 0 parts

Commit message: update,
Parts:
- added C?: C106,0805, Capacitor_SMD:C_0805_2012Metric_Pad1.15x1.40mm_HandSolder, symbol taobao-c:C106,0805
- added J? (x3): Conn_01x06, symbol Connector_Generic:Conn_01x06
- added J? (x2): Conn_01x05, symbol Connector_Generic:Conn_01x05
- added JP?: Jumper_2_Open, symbol Jumper:Jumper_2_Open
- added R? (x2): R121,0805, Resistor_SMD:R_0805_2012Metric_Pad1.15x1.40mm_HandSolder, symbol taobao-r:R121,0805
- added SW? (x2): microswitch_6_6_5, footprint-lib:microswitch_6_6_5, symbol taobao-components:microswitch_6_6_5
- added U?: SN65HVD232DR, Package_SO:SOIC-8-1EP_3.9x4.9mm_P1.27mm_EP2.29x3mm, symbol taobao-components:SN65HVD232DR
- added U?: TL431IDBZT, Package_TO_SOT_SMD:SOT-23, symbol taobao-components:TL431IDBZT
Connections:
- new net: JP?.1 (A), R?.2
- new net: J?.4 (Pin_4), R?.2, U?.1 (K), U?.2 (REF)
- new net +3V3: C?.1, J?.6 (Pin_6), R?.1, U?.3 (VCC)
- new net ADC_END: J?.5 (Pin_5)
- new net BUTTON_1: SW?.2
- new net BUTTON_2: SW?.2
- new net CAN_H: J?.4 (Pin_4), J?.4 (Pin_4), R?.1, U?.7 (CANH)
- new net CAN_L: J?.3 (Pin_3), J?.3 (Pin_3), JP?.2 (B), U?.6 (CANL)
- new net CAN_RX: U?.4 (R)
- new net CAN_TX: U?.1 (D)
- new net GND: C?.2, J?.1 (Pin_1), J?.4 (Pin_4), J?.5 (Pin_5), J?.5 (Pin_5), J?.5 (Pin_5), J?.5 (Pin_5), J?.6 (Pin_6), J?.6 (Pin_6), SW?.1, SW?.1, U?.2 (GND), U?.3 (A)
- new net MT6816_AUX_CS: J?.1 (Pin_1), J?.1 (Pin_1)
- new net SPI1_MISO: J?.2 (Pin_2), J?.2 (Pin_2)
- new net SPI1_MOSI: J?.3 (Pin_3), J?.3 (Pin_3)
- new net SPI1_SCK: J?.4 (Pin_4)
- new net SWCLK: J?.2 (Pin_2)
- new net SWDIO: J?.3 (Pin_3)
- new net VCC: J?.1 (Pin_1), J?.1 (Pin_1), J?.2 (Pin_2), J?.2 (Pin_2)

Commit message: update,
Parts:
- gave numbers to parts that had none: 13
Changed lines of the file:
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@@
   (symbol (lib_id "taobao-components:SN65HVD232DR") (at 76.2 118.11 0) (unit 1)
     (in_bom yes) (on_board yes) (fields_autoplaced)
-    (property "Reference" "U?" (id 0) (at 76.2 106.68 0))
+    (property "Reference" "U5" (id 0) (at 76.2 106.68 0))
     (property "Value" "SN65HVD232DR" (id 1) (at 76.2 109.22 0))
     (property "Footprint" "Package_SO:SOIC-8-1EP_3.9x4.9mm_P1.27mm_EP2.29x3mm" (id 2) (at 76.2 118.11 0)
@@
   (symbol (lib_id "Connector_Generic:Conn_01x06") (at 105.41 34.29 180) (unit 1)
     (in_bom yes) (on_board yes) (fields_autoplaced)
-    (property "Reference" "J?" (id 0) (at 105.41 20.32 0))
+    (property "Reference" "J2" (id 0) (at 105.41 20.32 0))
     (property "Value" "Conn_01x06" (id 1) (at 105.41 22.86 0))
     (property "Footprint" "" (id 2) (at 105.41 34.29 0)
@@
   (symbol (lib_id "Jumper:Jumper_2_Open") (at 72.39 90.17 0) (unit 1)
     (in_bom yes) (on_board yes) (fields_autoplaced)
-    (property "Reference" "JP?" (id 0) (at 72.39 83.82 0))
+    (property "Reference" "JP1" (id 0) (at 72.39 83.82 0))
     (property "Value" "Jumper_2_Open" (id 1) (at 72.39 86.36 0))
     (property "Footprint" "" (id 2) (at 72.39 90.17 0)
@@
   (symbol (lib_id "Connector_Generic:Conn_01x05") (at 105.41 71.12 180) (unit 1)
     (in_bom yes) (on_board yes) (fields_autoplaced)
-    (property "Reference" "J?" (id 0) (at 105.41 59.69 0))
+    (property "Reference" "J5" (id 0) (at 105.41 59.69 0))
     (property "Value" "Conn_01x05" (id 1) (at 105.41 62.23 0))
     (property "Footprint" "" (id 2) (at 105.41 71.12 0)
@@
   (symbol (lib_id "Connector_Generic:Conn_01x05") (at 22.86 33.02 180) (unit 1)
     (in_bom yes) (on_board yes) (fields_autoplaced)
-    (property "Reference" "J?" (id 0) (at 22.86 21.59 0))
+    (property "Reference" "J1" (id 0) (at 22.86 21.59 0))
     (property "Value" "Conn_01x05" (id 1) (at 22.86 24.13 0))
     (property "Footprint" "" (id 2) (at 22.86 33.02 0)
@@
   (symbol (lib_id "Connector_Generic:Conn_01x06") (at 22.86 72.39 180) (unit 1)
     (in_bom yes) (on_board yes) (fields_autoplaced)
-    (property "Reference" "J?" (id 0) (at 22.86 58.42 0))
+    (property "Reference" "J4" (id 0) (at 22.86 58.42 0))
     (property "Value" "Conn_01x06" (id 1) (at 22.86 60.96 0))
     (property "Footprint" "" (id 2) (at 22.86 72.39 0)
@@
   (symbol (lib_id "Connector_Generic:Conn_01x06") (at 152.4 34.29 180) (unit 1)
     (in_bom yes) (on_board yes) (fields_autoplaced)
-    (property "Reference" "J?" (id 0) (at 152.4 20.32 0))
+    (property "Reference" "J3" (id 0) (at 152.4 20.32 0))
     (property "Value" "Conn_01x06" (id 1) (at 152.4 22.86 0))
     (property "Footprint" "" (id 2) (at 152.4 34.29 0)
@@
   (symbol (lib_id "taobao-components:microswitch_6_6_5") (at 165.1 88.9 0) (unit 1)
     (in_bom yes) (on_board yes) (fields_autoplaced)
-    (property "Reference" "SW?" (id 0) (at 165.1 81.28 0))
+    (property "Reference" "SW2" (id 0) (at 165.1 81.28 0))
     (property "Value" "microswitch_6_6_5" (id 1) (at 165.1 83.82 0))
     (property "Footprint" "footprint-lib:microswitch_6_6_5" (id 2) (at 165.1 83.82 0)
@@
   (symbol (lib_id "taobao-r:R121,0805") (at 67.31 30.48 270) (unit 1)
     (in_bom yes) (on_board yes) (fields_autoplaced)
-    (property "Reference" "R?" (id 0) (at 68.5801 33.02 0)
+    (property "Reference" "R11" (id 0) (at 68.5801 33.02 0)
       (effects (font (size 1.27 1.27)) (justify left))
     )
@@
   (symbol (lib_id "taobao-components:microswitch_6_6_5") (at 165.1 77.47 0) (unit 1)
     (in_bom yes) (on_board yes) (fields_autoplaced)
-    (property "Reference" "SW?" (id 0) (at 165.1 69.85 0))
+    (property "Reference" "SW1" (id 0) (at 165.1 69.85 0))
     (property "Value" "microswitch_6_6_5" (id 1) (at 165.1 72.39 0))
     (property "Footprint" "footprint-lib:microswitch_6_6_5" (id 2) (at 165.1 72.39 0)
@@
   (symbol (lib_id "taobao-r:R121,0805") (at 55.88 90.17 90) (unit 1)
     (in_bom yes) (on_board yes) (fields_autoplaced)
-    (property "Reference" "R?" (id 0) (at 55.88 83.82 90))
+    (property "Reference" "R12" (id 0) (at 55.88 83.82 90))
     (property "Value" "R121,0805" (id 1) (at 55.88 86.36 90))
     (property "Footprint" "Resistor_SMD:R_0805_2012Metric_Pad1.15x1.40mm_HandSolder" (id 2) (at 55.88 90.17 0)
@@
   (symbol (lib_id "taobao-components:TL431IDBZT") (at 57.15 26.67 270) (unit 1)
     (in_bom yes) (on_board yes) (fields_autoplaced)
-    (property "Reference" "U?" (id 0) (at 54.61 25.3999 90)
+    (property "Reference" "U4" (id 0) (at 54.61 25.3999 90)
       (effects (font (size 1.27 1.27)) (justify right))
     )
@@
   (symbol (lib_id "taobao-c:C106,0805") (at 27.94 118.11 0) (unit 1)
     (in_bom yes) (on_board yes) (fields_autoplaced)
-    (property "Reference" "C?" (id 0) (at 30.48 116.8462 0)
+    (property "Reference" "C10" (id 0) (at 30.48 116.8462 0)
       (effects (font (size 1.27 1.27)) (justify left))
     )
