File: interface.kicad_sch (KiCad schematic)
At the start: 0 parts

Commit message: update,
Parts:
- added C?: C106,0805, Capacitor_SMD:C_0805_2012Metric_Pad1.15x1.40mm_HandSolder, symbol taobao-c:C106,0805
- added C? (x2): C104,0805, Capacitor_SMD:C_0805_2012Metric_Pad1.15x1.40mm_HandSolder, symbol taobao-c:C104,0805
- added R?: R103,0805, Resistor_SMD:R_0805_2012Metric_Pad1.15x1.40mm_HandSolder, symbol taobao-r:R103,0805
- added R?: R102,0805, Resistor_SMD:R_0805_2012Metric_Pad1.15x1.40mm_HandSolder, symbol taobao-r:R102,0805
- added U?: MT6816, symbol taobao-components:MT6816
Connections:
- new net: C?.2, R?.1, R?.2
- new net +3V3: C?.1, C?.1, U?.2 (HVPP), U?.4 (VDD)
- new net GND: C?.2, C?.2, R?.2, U?.5 (A_U)
- new net MT6816_CS: U?.1 (CSN)
- new net SPI1_MISO: U?.7 (Z_W)
- new net SPI1_MOSI: U?.8 (GND)
- new net SPI1_SCK: U?.6 (B_V)
- new net VCC: C?.1, R?.1

Commit message: update,
Parts:
- U?: footprint (none) -> JLC2KiCad_lib:MT6816CT-ACD; LCSC_PARTS (none) -> C879560
Changed lines of the file:
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@@
   (symbol (lib_id "taobao-c:C104,0805") (at 55.88 30.48 90) (unit 1)
     (in_bom yes) (on_board yes) (fields_autoplaced)
-    (property "Reference" "C?" (id 0) (at 55.8863 24.13 90))
-    (property "Value" "C104,0805" (id 1) (at 55.8863 26.67 90))
+    (property "Reference" "C?" (id 0) (at 55.8863 34.29 90))
+    (property "Value" "C104,0805" (id 1) (at 55.8863 36.83 90))
     (property "Footprint" "Capacitor_SMD:C_0805_2012Metric_Pad1.15x1.40mm_HandSolder" (id 2) (at 55.88 30.48 0)
       (effects (font (size 1.27 1.27)) hide)
@@
     (property "Reference" "U?" (id 0) (at 53.34 46.99 0))
     (property "Value" "MT6816" (id 1) (at 53.34 49.53 0))
-    (property "Footprint" "" (id 2) (at 53.34 58.42 0)
+    (property "Footprint" "JLC2KiCad_lib:MT6816CT-ACD" (id 2) (at 53.34 58.42 0)
       (effects (font (size 1.27 1.27)) hide)
     )
@@
       (effects (font (size 1.27 1.27)) hide)
     )
+    (property "Field4" "" (id 4) (at 53.34 58.42 0)
+      (effects (font (size 1.27 1.27)) hide)
+    )
+    (property "LCSC_PARTS" "C879560" (id 5) (at 53.34 58.42 0))
     (pin "1")
     (pin "2")

Commit message: update,
Parts:
- gave numbers to parts that had none: 6
Changed lines of the file:
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@@
     (stroke (width 0) (type default) (color 0 0 0 0))
   )
-  (image (at 223.52 31.75)
+  (image (at 177.8 82.55)
     (data
       iVBORw0KGgoAAAANSUhEUgAAAawAAAHjCAIAAADwpLxCAAAAA3NCSVQICAjb4U/gAAAgAElEQVR4
@@
   (symbol (lib_id "taobao-c:C106,0805") (at 55.88 22.86 90) (unit 1)
     (in_bom yes) (on_board yes) (fields_autoplaced)
-    (property "Reference" "C?" (id 0) (at 55.8863 16.51 90))
+    (property "Reference" "C24" (id 0) (at 55.8863 16.51 90))
     (property "Value" "C106,0805" (id 1) (at 55.8863 19.05 90))
     (property "Footprint" "Capacitor_SMD:C_0805_2012Metric_Pad1.15x1.40mm_HandSolder" (id 2) (at 55.88 22.86 0)
@@
   (symbol (lib_id "taobao-c:C104,0805") (at 55.88 30.48 90) (unit 1)
     (in_bom yes) (on_board yes) (fields_autoplaced)
-    (property "Reference" "C?" (id 0) (at 55.8863 34.29 90))
+    (property "Reference" "C25" (id 0) (at 55.8863 34.29 90))
     (property "Value" "C104,0805" (id 1) (at 55.8863 36.83 90))
     (property "Footprint" "Capacitor_SMD:C_0805_2012Metric_Pad1.15x1.40mm_HandSolder" (id 2) (at 55.88 30.48 0)
@@
   (symbol (lib_id "taobao-c:C104,0805") (at 123.19 53.34 90) (unit 1)
     (in_bom yes) (on_board yes) (fields_autoplaced)
-    (property "Reference" "C?" (id 0) (at 123.1963 46.99 90))
+    (property "Reference" "C26" (id 0) (at 123.1963 46.99 90))
     (property "Value" "C104,0805" (id 1) (at 123.1963 49.53 90))
     (property "Footprint" "Capacitor_SMD:C_0805_2012Metric_Pad1.15x1.40mm_HandSolder" (id 2) (at 123.19 53.34 0)
@@
   (symbol (lib_id "taobao-components:MT6816") (at 53.34 58.42 0) (unit 1)
     (in_bom yes) (on_board yes) (fields_autoplaced)
-    (property "Reference" "U?" (id 0) (at 53.34 46.99 0))
+    (property "Reference" "U8" (id 0) (at 53.34 46.99 0))
     (property "Value" "MT6816" (id 1) (at 53.34 49.53 0))
     (property "Footprint" "JLC2KiCad_lib:MT6816CT-ACD" (id 2) (at 53.34 58.42 0)
@@
   (symbol (lib_id "taobao-r:R103,0805") (at 123.19 40.64 90) (unit 1)
     (in_bom yes) (on_board yes) (fields_autoplaced)
-    (property "Reference" "R?" (id 0) (at 123.19 34.29 90))
+    (property "Reference" "R16" (id 0) (at 123.19 34.29 90))
     (property "Value" "R103,0805" (id 1) (at 123.19 36.83 90))
     (property "Footprint" "Resistor_SMD:R_0805_2012Metric_Pad1.15x1.40mm_HandSolder" (id 2) (at 123.19 40.64 0)
@@
   (symbol (lib_id "taobao-r:R102,0805") (at 143.51 40.64 90) (unit 1)
     (in_bom yes) (on_board yes) (fields_autoplaced)
-    (property "Reference" "R?" (id 0) (at 143.51 34.29 90))
+    (property "Reference" "R17" (id 0) (at 143.51 34.29 90))
     (property "Value" "R102,0805" (id 1) (at 143.51 36.83 90))
     (property "Footprint" "Resistor_SMD:R_0805_2012Metric_Pad1.15x1.40mm_HandSolder" (id 2) (at 143.51 40.64 0)
