File: drive.kicad_sch (KiCad schematic)
At the start: 0 parts

Commit message: update,
Parts:
- added C? (x4): C104,0805, Capacitor_SMD:C_0805_2012Metric_Pad1.15x1.40mm_HandSolder, symbol taobao-c:C104,0805
- added C?: C106,0805, Capacitor_SMD:C_0805_2012Metric_Pad1.15x1.40mm_HandSolder, symbol taobao-c:C106,0805
- added R? (x4): R102,0805, Resistor_SMD:R_0805_2012Metric_Pad1.15x1.40mm_HandSolder, symbol taobao-r:R102,0805
- added R?: NTC_10K,0805, Resistor_SMD:R_0805_2012Metric_Pad1.15x1.40mm_HandSolder, symbol taobao-r:NTC_10K,0805
- added R? (x2): R100,1206, Resistor_SMD:R_0805_2012Metric_Pad1.15x1.40mm_HandSolder, symbol taobao-r:R100,1206
- added R?: R332,0805, Resistor_SMD:R_0805_2012Metric_Pad1.15x1.40mm_HandSolder, symbol taobao-r:R332,0805
- added U? (x2): TB67H450FNG, Package_SO:HSOP-8-1EP_3.9x4.9mm_P1.27mm_EP2.41x3.1mm_ThermalVias, symbol taobao-components:TB67H450FNG
Connections:
- new net: C?.1, R?.1, R?.2 (x2)
- new net: R?.1, U?.7 (LSS) (x2)
- new net: C?.1, R?.2 (x2)
- new net +3V3: R?.1
- new net GND: C?.2, C?.2, C?.2, C?.2, C?.2, R?.2, R?.2, R?.2, U?.1 (GND), U?.1 (GND), U?.9 (EP), U?.9 (EP)
- new net IN_AM: U?.2 (IN2), U?.2 (IN2)
- new net IN_AP: U?.3 (IN1), U?.3 (IN1)
- new net IN_PWM_A: R?.1
- new net IN_PWM_B: R?.1
- new net OUT_A_N: U?.8 (OUT2)
- new net OUT_A_P: U?.6 (OUT1)
- new net OUT_B_N: U?.8 (OUT2)
- new net OUT_B_P: U?.6 (OUT1)
- new net TEMP: C?.1, R?.1, R?.2
- new net VCC: U?.5 (VCC), U?.5 (VCC)
- new net VREF_A: U?.4 (VREF), U?.4 (VREF)

Commit message: update,
Parts:
- U? (x2): PRICE (none) -> 3; TAOBAO (none) -> https://item.taobao.com/item.htm?spm=a230r.1.14.68.5d9f7a9b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
Other:
- moved on the sheet: C?, R?, U?

Commit message: update,
Parts:
- gave numbers to parts that had none: 4
Changed lines of the file:
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@@
   (symbol (lib_id "taobao-r:R102,0805") (at 33.02 31.75 90) (unit 1)
     (in_bom yes) (on_board yes) (fields_autoplaced)
-    (property "Reference" "R?" (id 0) (at 33.02 25.4 90))
+    (property "Reference" "R1" (id 0) (at 33.02 25.4 90))
     (property "Value" "R102,0805" (id 1) (at 33.02 27.94 90))
     (property "Footprint" "Resistor_SMD:R_0805_2012Metric_Pad1.15x1.40mm_HandSolder" (id 2) (at 33.02 31.75 0)
@@
   (symbol (lib_id "taobao-c:C104,0805") (at 40.64 38.1 0) (unit 1)
     (in_bom yes) (on_board yes) (fields_autoplaced)
-    (property "Reference" "C?" (id 0) (at 43.18 36.8362 0)
+    (property "Reference" "C1" (id 0) (at 43.18 36.8362 0)
       (effects (font (size 1.27 1.27)) (justify left))
     )
@@
   (symbol (lib_id "taobao-r:R102,0805") (at 46.99 31.75 90) (unit 1)
     (in_bom yes) (on_board yes) (fields_autoplaced)
-    (property "Reference" "R?" (id 0) (at 46.99 25.4 90))
+    (property "Reference" "R2" (id 0) (at 46.99 25.4 90))
     (property "Value" "R102,0805" (id 1) (at 46.99 27.94 90))
     (property "Footprint" "Resistor_SMD:R_0805_2012Metric_Pad1.15x1.40mm_HandSolder" (id 2) (at 46.99 31.75 0)
@@
   (symbol (lib_id "taobao-c:C104,0805") (at 57.15 38.1 0) (unit 1)
     (in_bom yes) (on_board yes) (fields_autoplaced)
-    (property "Reference" "C?" (id 0) (at 59.69 36.8362 0)
+    (property "Reference" "C2" (id 0) (at 59.69 36.8362 0)
       (effects (font (size 1.27 1.27)) (justify left))
     )

Commit message: update,
Parts:
- gave numbers to parts that had none: 4
Changed lines of the file:
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@@
   (symbol (lib_id "taobao-r:R102,0805") (at 33.02 68.58 90) (unit 1)
     (in_bom yes) (on_board yes) (fields_autoplaced)
-    (property "Reference" "R?" (id 0) (at 33.02 62.23 90))
+    (property "Reference" "R6" (id 0) (at 33.02 62.23 90))
     (property "Value" "R102,0805" (id 1) (at 33.02 64.77 90))
     (property "Footprint" "Resistor_SMD:R_0805_2012Metric_Pad1.15x1.40mm_HandSolder" (id 2) (at 33.02 68.58 0)
@@
   (symbol (lib_id "taobao-c:C104,0805") (at 40.64 74.93 0) (unit 1)
     (in_bom yes) (on_board yes) (fields_autoplaced)
-    (property "Reference" "C?" (id 0) (at 43.18 73.6662 0)
+    (property "Reference" "C4" (id 0) (at 43.18 73.6662 0)
       (effects (font (size 1.27 1.27)) (justify left))
     )
@@
   (symbol (lib_id "taobao-c:C104,0805") (at 57.15 74.93 0) (unit 1)
     (in_bom yes) (on_board yes) (fields_autoplaced)
-    (property "Reference" "C?" (id 0) (at 59.69 73.6662 0)
+    (property "Reference" "C5" (id 0) (at 59.69 73.6662 0)
       (effects (font (size 1.27 1.27)) (justify left))
     )
@@
   (symbol (lib_id "taobao-r:R102,0805") (at 46.99 68.58 90) (unit 1)
     (in_bom yes) (on_board yes) (fields_autoplaced)
-    (property "Reference" "R?" (id 0) (at 46.99 62.23 90))
+    (property "Reference" "R7" (id 0) (at 46.99 62.23 90))
     (property "Value" "R102,0805" (id 1) (at 46.99 64.77 90))
     (property "Footprint" "Resistor_SMD:R_0805_2012Metric_Pad1.15x1.40mm_HandSolder" (id 2) (at 46.99 68.58 0)

Commit message: update,
Parts:
- U1, U2: renamed from U?; footprint Package_SO:HSOP-8-1EP_3.9x4.9mm_P1.27mm_EP2.41x3.1mm_ThermalVias -> LCSC:TB67H450FNG,EL; LCSC Part (none) -> C129353
Changed lines of the file:
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@@
   (symbol (lib_name "TB67H450FNG_1") (lib_id "taobao-components:TB67H450FNG") (at 101.6 91.44 0) (unit 1)
     (in_bom yes) (on_board yes) (fields_autoplaced)
-    (property "Reference" "U?" (id 0) (at 101.6 78.74 0))
+    (property "Reference" "U2" (id 0) (at 101.6 78.74 0))
     (property "Value" "TB67H450FNG" (id 1) (at 101.6 81.28 0))
-    (property "Footprint" "Package_SO:HSOP-8-1EP_3.9x4.9mm_P1.27mm_EP2.41x3.1mm_ThermalVias" (id 2) (at 101.6 105.41 0)
+    (property "Footprint" "LCSC:TB67H450FNG,EL" (id 2) (at 101.6 105.41 0)
       (effects (font (size 1.27 1.27)) hide)
     )
@@
     (property "PRICE" "3" (id 4) (at 101.6 91.44 0))
     (property "TAOBAO" "https://item.taobao.com/item.htm?spm=a230r.1.14.68.5d9f7a9buKNpPG&id=611742699273&ns=1&abbucket=19#detail" (id 5) (at 101.6 91.44 0))
+    (property "LCSC Part" "C129353" (id 6) (at 101.6 91.44 0))
     (pin "1")
     (pin "2")
@@
   (symbol (lib_id "taobao-components:TB67H450FNG") (at 101.6 54.61 0) (unit 1)
     (in_bom yes) (on_board yes) (fields_autoplaced)
-    (property "Reference" "U?" (id 0) (at 101.6 41.91 0))
+    (property "Reference" "U1" (id 0) (at 101.6 41.91 0))
     (property "Value" "TB67H450FNG" (id 1) (at 101.6 44.45 0))
-    (property "Footprint" "Package_SO:HSOP-8-1EP_3.9x4.9mm_P1.27mm_EP2.41x3.1mm_ThermalVias" (id 2) (at 101.6 68.58 0)
+    (property "Footprint" "LCSC:TB67H450FNG,EL" (id 2) (at 101.6 68.58 0)
       (effects (font (size 1.27 1.27)) hide)
     )
     (property "Datasheet" "" (id 3) (at 101.6 54.61 0)
-      (effects (font (size 1.27 1.27)) hide)
-    )
-    (property "Field4" "" (id 4) (at 101.6 54.61 0)
       (effects (font (size 1.27 1.27)) hide)
     )
@@
       (effects (font (size 1.27 1.27)) hide)
     )
+    (property "LCSC Part" "C129353" (id 7) (at 101.6 54.61 0))
     (pin "1")
     (pin "2")

Commit message: update,
Parts:
- gave numbers to parts that had none: 3
Changed lines of the file:
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@@
   (symbol (lib_id "taobao-r:NTC_10K,0805") (at 171.45 34.29 0) (unit 1)
     (in_bom yes) (on_board yes) (fields_autoplaced)
-    (property "Reference" "R?" (id 0) (at 173.99 33.0199 0)
+    (property "Reference" "R4" (id 0) (at 173.99 33.0199 0)
       (effects (font (size 1.27 1.27)) (justify left))
     )
@@
     (pin "2")
   )
-  (symbol (lib_name "TB67H450FNG_1") (lib_id "taobao-components:TB67H450FNG") (at 101.6 91.44 0) (unit 1)
+  (symbol (lib_id "taobao-components:TB67H450FNG") (at 101.6 91.44 0) (unit 1)
     (in_bom yes) (on_board yes) (fields_autoplaced)
     (property "Reference" "U2" (id 0) (at 101.6 78.74 0))
@@
     )
     (property "PRICE" "3" (id 4) (at 101.6 91.44 0))
-    (property "TAOBAO" "https://item.taobao.com/item.htm?spm=a230r.1.14.68.5d9f7a9buKNpPG&id=611742699273&ns=1&abbucket=19#detail" (id 5) (at 101.6 91.44 0))
+    (property "TAOBAO" "https://item.taobao.com/item.htm?spm=a230r.1.14.68.5d9f7a9buKNpPG&id=611742699273&ns=1&abbucket=19#detail" (id 5) (at 101.6 91.44 0)
+      (effects (font (size 1.27 1.27)) hide)
+    )
     (property "LCSC Part" "C129353" (id 6) (at 101.6 91.44 0))
     (pin "1")
@@
   (symbol (lib_id "taobao-r:R332,0805") (at 171.45 50.8 0) (unit 1)
     (in_bom yes) (on_board yes) (fields_autoplaced)
-    (property "Reference" "R?" (id 0) (at 173.99 49.5299 0)
+    (property "Reference" "R5" (id 0) (at 173.99 49.5299 0)
       (effects (font (size 1.27 1.27)) (justify left))
     )
@@
   (symbol (lib_id "taobao-c:C106,0805") (at 157.48 50.8 0) (unit 1)
     (in_bom yes) (on_board yes) (fields_autoplaced)
-    (property "Reference" "C?" (id 0) (at 160.02 49.5362 0)
-      (effects (font (size 1.27 1.27)) (justify left))
-    )
+    (property "Reference" "C3" (id 0) (at 160.02 49.5362 0)
+      (effects (font (size 1.27 1.27)) (justify left))
+    )

Commit message: update,
Parts:
- gave numbers to parts that had none: 2
Changed lines of the file:
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@@
   (symbol (lib_id "taobao-r:R100,1206") (at 134.62 54.61 90) (unit 1)
     (in_bom yes) (on_board yes) (fields_autoplaced)
-    (property "Reference" "R?" (id 0) (at 134.62 48.26 90))
+    (property "Reference" "R3" (id 0) (at 134.62 48.26 90))
     (property "Value" "R100,1206" (id 1) (at 134.62 50.8 90))
     (property "Footprint" "Resistor_SMD:R_0805_2012Metric_Pad1.15x1.40mm_HandSolder" (id 2) (at 134.62 54.61 0)
@@
   (symbol (lib_id "taobao-r:R100,1206") (at 134.62 91.44 90) (unit 1)
     (in_bom yes) (on_board yes) (fields_autoplaced)
-    (property "Reference" "R?" (id 0) (at 134.62 85.09 90))
+    (property "Reference" "R8" (id 0) (at 134.62 85.09 90))
     (property "Value" "R100,1206" (id 1) (at 134.62 87.63 90))
     (property "Footprint" "Resistor_SMD:R_0805_2012Metric_Pad1.15x1.40mm_HandSolder" (id 2) (at 134.62 91.44 0)
