File: MCU.kicad_sch (KiCad schematic)
At the start: 0 parts

Commit message: update,
Parts:
- added C? (x4): C104,0805, Capacitor_SMD:C_0805_2012Metric_Pad1.15x1.40mm_HandSolder, symbol taobao-c:C104,0805
- added R? (x2): R103,0805, Resistor_SMD:R_0805_2012Metric_Pad1.15x1.40mm_HandSolder, symbol taobao-r:R103,0805
- added U? (x2): STM32F103CBT6, Package_QFP:LQFP-48_7x7mm_P0.5mm, symbol taobao-components:STM32F103CBT6
- added Y?: O_12M,3225, footprint-lib:OSC_3225, symbol taobao-osc:O_12M,3225
Connections:
- new net: R?.1, U?.44 (BOOT0)
- new net: U?.5 (PD0-OSC-IN), Y?.1
- new net: U?.6 (PD1-OSC-OUT), Y?.3
- new net: C?.2, R?.1, U?.7 (NRST)
- new net +3V3: C?.1, C?.1, C?.1, R?.2, U?.1 (VBAT), U?.24 (VDD_1), U?.36 (VDD_2), U?.48 (VDD_3), U?.9 (VDDA)
- new net ADC_ENC: U?.16 (PA6)
- new net BUTTON_1: U?.30 (PB12)
- new net BUTTON_2: U?.20 (PB2)
- new net CAN_RX: U?.26 (PB8)
- new net CAN_TX: U?.27 (PB9)
- new net GND: C?.1, C?.2, C?.2, C?.2, R?.2, U?.23 (VSS_1), U?.35 (VSS_2), U?.47 (VSS_3), U?.8 (VSSA), Y?.2
- new net IN_AM: U?.14 (PA4)
- new net IN_AP: U?.15 (PA5)
- new net IN_BM: U?.12 (PA2)
- new net IN_BP: U?.13 (PA3)
- new net IN_PWM_A: U?.29 (PB11)
- new net IN_PWM_B: U?.28 (PB10)
- new net MT6816_AUX_CS: U?.17 (PA7)
- new net MT6816_CS: U?.38 (PA15)
- new net OLED_DC: U?.29 (PB11)
- new net OLED_RES: U?.30 (PB12)
- new net PA_10: U?.31 (PB13)
- new net PB0: U?.18 (PB0)
- new net PB1: U?.19 (PB1)
- new net PC13: U?.2 (PC13-TAMPER-RTC)
- new net PC14: U?.3 (PC14-OSC32-IN)
- new net PC15: U?.4 (PC15-OSC32-OUT)
- new net POWER_U: U?.10 (PA0_WKUP)
- new net SPI1_MISO: U?.22 (PB4)
- new net SPI1_MOSI: U?.23 (PB5)
- new net SPI1_SCK: U?.21 (PB3)
- new net SPI2_MISO: U?.32 (PB14)
- new net SPI2_MOSI: U?.33 (PB15)
- new net SPI2_SCK: U?.31 (PB13)
- new net SWCLK: U?.37 (PA14)
- new net SWDIO: U?.34 (PA13)
- new net TEMP: U?.11 (PA1)
- new net UART1_RX: U?.25 (PB7)
- new net UART1_TX: U?.24 (PB6)
- new net USB_DM: U?.32 (PB14)
- new net USB_DP: U?.33 (PB15)

Commit message: update,
Parts:
- gave numbers to parts that had none: 5
Changed lines of the file:
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@@
     (stroke (width 0) (type default) (color 0 0 0 0))
   )
-  (image (at 350.52 43.18)
+  (image (at 270.51 41.91)
     (data
       iVBORw0KGgoAAAANSUhEUgAABWYAAALrCAIAAADyW8lYAAAAA3NCSVQICAjb4U/gAAAgAElEQVR4
@@
   (symbol (lib_id "taobao-components:STM32F103CBT6") (at 76.2 62.23 0) (unit 1)
     (in_bom yes) (on_board yes) (fields_autoplaced)
-    (property "Reference" "U?" (id 0) (at 76.2 15.24 0))
+    (property "Reference" "U3" (id 0) (at 76.2 15.24 0))
     (property "Value" "STM32F103CBT6" (id 1) (at 76.2 17.78 0))
     (property "Footprint" "Package_QFP:LQFP-48_7x7mm_P0.5mm" (id 2) (at 76.2 96.52 0)
@@
   (symbol (lib_id "taobao-c:C104,0805") (at 109.22 86.36 180) (unit 1)
     (in_bom yes) (on_board yes) (fields_autoplaced)
-    (property "Reference" "C?" (id 0) (at 111.76 85.0835 0)
+    (property "Reference" "C9" (id 0) (at 111.76 85.0835 0)
       (effects (font (size 1.27 1.27)) (justify right))
     )
@@
   (symbol (lib_id "taobao-r:R103,0805") (at 116.84 82.55 90) (unit 1)
     (in_bom yes) (on_board yes) (fields_autoplaced)
-    (property "Reference" "R?" (id 0) (at 116.84 76.2 90))
+    (property "Reference" "R10" (id 0) (at 116.84 76.2 90))
     (property "Value" "R103,0805" (id 1) (at 116.84 78.74 90))
     (property "Footprint" "Resistor_SMD:R_0805_2012Metric_Pad1.15x1.40mm_HandSolder" (id 2) (at 116.84 82.55 0)
@@
   (symbol (lib_id "taobao-r:R103,0805") (at 116.84 74.93 90) (unit 1)
     (in_bom yes) (on_board yes) (fields_autoplaced)
-    (property "Reference" "R?" (id 0) (at 116.84 68.58 90))
+    (property "Reference" "R9" (id 0) (at 116.84 68.58 90))
     (property "Value" "R103,0805" (id 1) (at 116.84 71.12 90))
     (property "Footprint" "Resistor_SMD:R_0805_2012Metric_Pad1.15x1.40mm_HandSolder" (id 2) (at 116.84 74.93 0)
@@
   (symbol (lib_id "taobao-osc:O_12M,3225") (at 34.29 85.09 270) (unit 1)
     (in_bom yes) (on_board yes) (fields_autoplaced)
-    (property "Reference" "Y?" (id 0) (at 36.83 83.8199 90)
+    (property "Reference" "Y1" (id 0) (at 36.83 83.8199 90)
       (effects (font (size 1.27 1.27)) (justify left))
     )

Commit message: update,
Parts:
- U3: footprint Package_QFP:LQFP-48_7x7mm_P0.5mm -> LCSC:STM32F103CBT6TR
- U3: renamed from U?; footprint Package_QFP:LQFP-48_7x7mm_P0.5mm -> LCSC:STM32F103CBT6TR; LCSC (none) -> https://lcsc.com/product-detail/New-Arrivals_STMicroelectro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
- gave numbers to parts that had none: 3
Changed lines of the file:
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@@
   (symbol (lib_id "taobao-c:C104,0805") (at 161.29 29.21 0) (unit 1)
     (in_bom yes) (on_board yes) (fields_autoplaced)
-    (property "Reference" "C?" (id 0) (at 163.83 27.9462 0)
+    (property "Reference" "C6" (id 0) (at 163.83 27.9462 0)
       (effects (font (size 1.27 1.27)) (justify left))
     )
@@
     (property "Reference" "U3" (id 0) (at 76.2 15.24 0))
     (property "Value" "STM32F103CBT6" (id 1) (at 76.2 17.78 0))
-    (property "Footprint" "Package_QFP:LQFP-48_7x7mm_P0.5mm" (id 2) (at 76.2 96.52 0)
+    (property "Footprint" "LCSC:STM32F103CBT6TR" (id 2) (at 76.2 96.52 0)
       (effects (font (size 1.27 1.27)) hide)
     )
@@
   (symbol (lib_id "taobao-c:C104,0805") (at 182.88 29.21 0) (unit 1)
     (in_bom yes) (on_board yes) (fields_autoplaced)
-    (property "Reference" "C?" (id 0) (at 185.42 27.9462 0)
+    (property "Reference" "C8" (id 0) (at 185.42 27.9462 0)
       (effects (font (size 1.27 1.27)) (justify left))
     )
@@
   (symbol (lib_name "STM32F103CBT6_1") (lib_id "taobao-components:STM32F103CBT6") (at 175.26 80.01 0) (unit 2)
     (in_bom yes) (on_board yes) (fields_autoplaced)
-    (property "Reference" "U?" (id 0) (at 175.5775 62.23 0))
+    (property "Reference" "U3" (id 0) (at 175.5775 62.23 0))
     (property "Value" "STM32F103CBT6" (id 1) (at 175.5775 64.77 0))
-    (property "Footprint" "Package_QFP:LQFP-48_7x7mm_P0.5mm" (id 2) (at 175.26 114.3 0)
+    (property "Footprint" "LCSC:STM32F103CBT6TR" (id 2) (at 175.26 114.3 0)
       (effects (font (size 1.27 1.27)) hide)
     )
     (property "Datasheet" "" (id 3) (at 175.26 114.3 0)
+      (effects (font (size 1.27 1.27)) hide)
+    )
+    (property "LCSC" "https://lcsc.com/product-detail/New-Arrivals_STMicroelectronics-STM32F103CBT6TR_C279569.html" (id 4) (at 175.26 80.01 0)
       (effects (font (size 1.27 1.27)) hide)
     )
@@
   (symbol (lib_id "taobao-c:C104,0805") (at 172.72 29.21 0) (unit 1)
     (in_bom yes) (on_board yes) (fields_autoplaced)
-    (property "Reference" "C?" (id 0) (at 175.26 27.9462 0)
+    (property "Reference" "C7" (id 0) (at 175.26 27.9462 0)
       (effects (font (size 1.27 1.27)) (justify left))
     )
