File: power.kicad_sch (KiCad schematic)
At the start: 0 parts

Commit message: update,
Parts:
- added C? (x2): C106,0805, Capacitor_SMD:C_0805_2012Metric_Pad1.15x1.40mm_HandSolder, symbol taobao-c:C106,0805
- added C? (x9): C106,50v,1206, Capacitor_SMD:C_1206_3216Metric_Pad1.42x1.75mm_HandSolder, symbol taobao-c:C106,50v,1206
- added C? (x4): C104,0805, Capacitor_SMD:C_0805_2012Metric_Pad1.15x1.40mm_HandSolder, symbol taobao-c:C104,0805
- added C?: C103,0805, Capacitor_SMD:C_0805_2012Metric_Pad1.15x1.40mm_HandSolder, symbol taobao-c:C103,0805
- added C?: C100pf,0805, Capacitor_SMD:C_0805_2012Metric_Pad1.15x1.40mm_HandSolder, symbol taobao-c:C100pf,0805
- added D? (x2): SD_1N5819_SS14, symbol taobao-sd:SD_1N5819_SS14
- added D?: SMBJ28CA, Diode_SMD:D_SMB, symbol taobao-d:SMBJ28CA
- added D?: SS54, Diode_SMD:D_SMC, symbol taobao-d:SS54
- added L?: L_6.8uH, symbol taobao-l:L_6.8uH
- added R?: R182,0805, Resistor_SMD:R_0805_2012Metric_Pad1.15x1.40mm_HandSolder, symbol taobao-r:R182,0805
- added R?: R103,0805, Resistor_SMD:R_0805_2012Metric_Pad1.15x1.40mm_HandSolder, symbol taobao-r:R103,0805
- added R?: R105,0805, Resistor_SMD:R_0805_2012Metric_Pad1.15x1.40mm_HandSolder, symbol taobao-r:R105,0805
- added U?: LP2992, symbol taobao-components:LP2992
- added U?: ME3116, symbol taobao-components:ME3116
Connections:
- new net: C?.1, C?.1, U?.1 (BS)
- new net: C?.2, C?.2, D?.1 (K), L?.1, U?.6 (SW)
- new net: C?.1, D?.1 (K), R?.2, U?.5 (IN)
- new net: C?.2, R?.1, R?.2, U?.3 (FB)
- new net: C?.1, U?.4 (BYPASS)
- new net: R?.1, U?.4 (EN)
- new net +3V3: C?.1, C?.1, U?.5 (VOUT)
- new net +5V: C?.1, C?.1, C?.2, L?.2, R?.1, U?.1 (VIN), U?.3 (ON_OFF)
- new net +DC_IN: D?.2 (A)
- new net GND: C?.1, C?.2, C?.2, C?.2, C?.2, C?.2, C?.2, C?.2, C?.2, C?.2, C?.2, C?.2, C?.2, C?.2, D?.1 (A1), D?.2 (A), R?.2, U?.2 (GND), U?.2 (GND)
- new net VCC: C?.1, C?.1, C?.1, C?.1, C?.1, C?.1, C?.1, C?.1, D?.1 (K), D?.2 (A), D?.2 (A2)

Commit message: update,
Parts:
- U?: footprint (none) -> LCSC:LP2992IM5-3.3_NOPB; LCSC (none) -> https://lcsc.com/product-detail/Linear-Voltage-Regulators-L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
- U?: footprint (none) -> LCSC:ME3116AM6G
Changed lines of the file:
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@@
     (property "Reference" "U?" (id 0) (at 53.34 68.58 0))
     (property "Value" "LP2992" (id 1) (at 53.34 71.12 0))
-    (property "Footprint" "" (id 2) (at 56.515 83.82 0)
+    (property "Footprint" "LCSC:LP2992IM5-3.3_NOPB" (id 2) (at 56.515 83.82 0)
       (effects (font (size 1.27 1.27)) hide)
     )
     (property "Datasheet" "" (id 3) (at 56.515 83.82 0)
+      (effects (font (size 1.27 1.27)) hide)
+    )
+    (property "LCSC" "https://lcsc.com/product-detail/Linear-Voltage-Regulators-LDO_Texas-Instruments-LP2992IM5-2-5-NOPB_C133799.html" (id 4) (at 53.34 83.82 0)
       (effects (font (size 1.27 1.27)) hide)
     )
@@
     (property "Reference" "U?" (id 0) (at 144.78 69.85 0))
     (property "Value" "ME3116" (id 1) (at 144.78 72.39 0))
-    (property "Footprint" "" (id 2) (at 144.78 81.28 0)
-      (effects (font (size 1.27 1.27)) hide)
-    )
+    (property "Footprint" "LCSC:ME3116AM6G" (id 2) (at 144.78 81.28 0)
+      (effects (font (size 1.27 1.27)) hide)
+    )

Commit message: update,
Parts:
- removed C? (x4): C106,50v,1206, Capacitor_SMD:C_1206_3216Metric_Pad1.42x1.75mm_HandSolder, symbol taobao-c:C106,50v,1206
- gave numbers to parts that had none: 20

Commit message: update,
Parts:
- gave numbers to parts that had none: 1
Changed lines of the file:
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@@
   (symbol (lib_id "taobao-c:C103,0805") (at 78.74 91.44 90) (unit 1)
     (in_bom yes) (on_board yes) (fields_autoplaced)
-    (property "Reference" "C?" (id 0) (at 78.7463 85.09 90))
+    (property "Reference" "C23" (id 0) (at 78.7463 85.09 90))
     (property "Value" "C103,0805" (id 1) (at 78.7463 87.63 90))
     (property "Footprint" "Capacitor_SMD:C_0805_2012Metric_Pad1.15x1.40mm_HandSolder" (id 2) (at 78.74 91.44 0)

Commit message: update,
Parts:
- gave numbers to parts that had none: 2
Changed lines of the file:
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@@
   (symbol (lib_id "taobao-c:C104,0805") (at 72.39 80.01 0) (unit 1)
     (in_bom yes) (on_board yes) (fields_autoplaced)
-    (property "Reference" "C?" (id 0) (at 74.93 78.7462 0)
+    (property "Reference" "C21" (id 0) (at 74.93 78.7462 0)
       (effects (font (size 1.27 1.27)) (justify left))
     )
@@
   (symbol (lib_id "taobao-c:C106,0805") (at 80.01 80.01 0) (unit 1)
     (in_bom yes) (on_board yes) (fields_autoplaced)
-    (property "Reference" "C?" (id 0) (at 82.55 78.7462 0)
-      (effects (font (size 1.27 1.27)) (justify left))
-    )
+    (property "Reference" "C22" (id 0) (at 82.55 78.7462 0)
+      (effects (font (size 1.27 1.27)) (justify left))
+    )

Commit message: update,
Parts:
- D3, D4: footprint (none) -> Diode_SMD:D_SMA
Changed lines of the file:
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@@
     (property "Reference" "D4" (id 0) (at 172.593 86.36 0))
     (property "Value" "SD_1N5819_SS14" (id 1) (at 172.593 88.9 0))
-    (property "Footprint" "" (id 2) (at 172.72 92.71 90)
+    (property "Footprint" "Diode_SMD:D_SMA" (id 2) (at 172.72 92.71 90)
       (effects (font (size 1.27 1.27)) hide)
     )
@@
     (property "Reference" "D3" (id 0) (at 172.593 72.39 0))
     (property "Value" "SD_1N5819_SS14" (id 1) (at 172.593 74.93 0))
-    (property "Footprint" "" (id 2) (at 172.72 78.74 90)
-      (effects (font (size 1.27 1.27)) hide)
-    )
+    (property "Footprint" "Diode_SMD:D_SMA" (id 2) (at 172.72 78.74 90)
+      (effects (font (size 1.27 1.27)) hide)
+    )
