File: 42-stepper-motor-driver-tryout.kicad_pcb (KiCad board)
At the start: 2 copper layers, 42 x 42 mm, 4 parts

Commit message: update,
Parts:
- added D1: SS54, Diode_SMD:D_SMC, F.Cu at (95.0, 48.0)
- added D2: SMBJ28CA, Diode_SMD:D_SMB, F.Cu at (93.8, 54.6)
- added D3: SD_1N5819_SS14, Diode_SMD:D_SMA, F.Cu at (102.0, 54.1)
- added D4: SD_1N5819_SS14, Diode_SMD:D_SMA, F.Cu at (104.5, 46.4)
- added SW1: microswitch_6_6_5, footprint-lib:microswitch_6_6_5, F.Cu at (93.9, 36.6)
- added SW2: microswitch_6_6_5, footprint-lib:microswitch_6_6_5, F.Cu at (93.9, 29.4)
- added U1: TB67H450FNG, LCSC:TB67H450FNG,EL, F.Cu at (127.7, 48.4)
- added U2: TB67H450FNG, LCSC:TB67H450FNG,EL, F.Cu at (121.1, 48.4)
- added U3: STM32F103CBT6, LCSC:STM32F103CBT6TR, F.Cu at (125.2, 31.4)
- added U4: TL431IDBZT, Package_TO_SOT_SMD:SOT-23, F.Cu at (100.7, 34.6)
- added U5: SN65HVD232DR, Package_SO:SOIC-8-1EP_3.9x4.9mm_P1.27mm_EP2.29x3mm, F.Cu at (102.5, 29.1)
- added U6: ME3116, LCSC:ME3116AM6G, F.Cu at (110.9, 46.3)
- added U7: LP2992, LCSC:LP2992IM5-3.3_NOPB, F.Cu at (108.3, 50.9)
- added Y1: O_12M,3225, footprint-lib:OSC_3225, F.Cu at (133.8, 28.6)
