File: hardware/42-stepper-motor-driver-tryout.kicad_sch (KiCad schematic)
At the start: 0 parts

Commit message: update,
Parts:
- added H1, H2, H3, H4: MountingHole, footprint-lib:MountingHole_2.7mm_M2.5,rpi_like, symbol Mechanical:MountingHole
Other:
- added sheet driver (driver.kicad_sch)
- added sheet ports (ports.kicad_sch)
- added sheet sensor (sensor.kicad_sch)
