File: hardware/node_mcu.kicad_sch (KiCad schematic)
At the start: 36 parts, among them Q1 S8050, Q2 S8050, SW1 microswitch_6_6_5, SW3 microswitch_6_6_5, U1 ESP-12E, U2 CH340G, U3 USB_Micro, U4 SPX3819M5-L

Commit message: update,
Parts:
- C10, C2, C4, C5, C6, C7, C8, C9: footprint Capacitor_SMD:C_0805_2012Metric_Pad1.15x1.40mm_HandSolder -> Capacitor_SMD:C_0805_2012Metric
- D1: footprint (none) -> Diode_SMD:D_SMA
- Q1, Q2: footprint Package_TO_SOT_THT:TO-92_Inline -> footprint-lib:S8050,J3Y,SOT23
- R1, R10, R11, R12, R13, R14, R7, R8, R9: footprint Resistor_SMD:R_0805_2012Metric_Pad1.15x1.40mm_HandSolder -> Resistor_SMD:R_0805_2012Metric
Connections:
- net GPIO0: now also Q2.C; no longer Q2.3 (C)
- net nRST: now also Q1.C; no longer Q1.3 (C)
- net at R13.2, U2.13 (~{DTR}): now also Q2.E; no longer Q2.1 (E)
- net at R14.2, U2.14 (~{RTS}): now also Q1.E; no longer Q1.1 (E)
- net at R13.1: now also Q1.B; no longer Q1.2 (B)
- net at R14.1: now also Q2.B; no longer Q2.2 (B)
Changed lines of the file:
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@@
       (effects (font (size 1.27 1.27)) (justify left))
     )
-    (property "Footprint" "Resistor_SMD:R_0805_2012Metric_Pad1.15x1.40mm_HandSolder" (id 2) (at 292.1 45.72 0)
+    (property "Footprint" "Resistor_SMD:R_0805_2012Metric" (id 2) (at 292.1 45.72 0)
       (effects (font (size 1.27 1.27)) hide)
     )
@@
       (effects (font (size 1.27 1.27)) (justify left))
     )
-    (property "Footprint" "Capacitor_SMD:C_0805_2012Metric_Pad1.15x1.40mm_HandSolder" (id 2) (at 57.15 129.54 0)
+    (property "Footprint" "Capacitor_SMD:C_0805_2012Metric" (id 2) (at 57.15 129.54 0)
       (effects (font (size 1.27 1.27)) hide)
     )
@@
       (effects (font (size 1.27 1.27)) (justify left))
     )
-    (property "Footprint" "Resistor_SMD:R_0805_2012Metric_Pad1.15x1.40mm_HandSolder" (id 2) (at 361.95 68.58 0)
+    (property "Footprint" "Resistor_SMD:R_0805_2012Metric" (id 2) (at 361.95 68.58 0)
       (effects (font (size 1.27 1.27)) hide)
     )
@@
       (effects (font (size 1.27 1.27)) (justify left))
     )
-    (property "Footprint" "Resistor_SMD:R_0805_2012Metric_Pad1.15x1.40mm_HandSolder" (id 2) (at 331.47 129.54 0)
+    (property "Footprint" "Resistor_SMD:R_0805_2012Metric" (id 2) (at 331.47 129.54 0)
       (effects (font (size 1.27 1.27)) hide)
     )
@@
     (property "Reference" "R10" (id 0) (at 204.47 125.73 90))
     (property "Value" "R471,0805" (id 1) (at 204.47 128.27 90))
-    (property "Footprint" "Resistor_SMD:R_0805_2012Metric_Pad1.15x1.40mm_HandSolder" (id 2) (at 204.47 132.08 0)
+    (property "Footprint" "Resistor_SMD:R_0805_2012Metric" (id 2) (at 204.47 132.08 0)
       (effects (font (size 1.27 1.27)) hide)
     )
@@
       (effects (font (size 1.27 1.27)) (justify left))
     )
-    (property "Footprint" "Capacitor_SMD:C_0805_2012Metric_Pad1.15x1.40mm_HandSolder" (id 2) (at 58.42 66.04 0)
+    (property "Footprint" "Capacitor_SMD:C_0805_2012Metric" (id 2) (at 58.42 66.04 0)
       (effects (font (size 1.27 1.27)) hide)
     )
@@
       (effects (font (size 1.27 1.27)) (justify left))
     )
-    (property "Footprint" "Resistor_SMD:R_0805_2012Metric_Pad1.15x1.40mm_HandSolder" (id 2) (at 292.1 64.77 0)
+    (property "Footprint" "Resistor_SMD:R_0805_2012Metric" (id 2) (at 292.1 64.77 0)
       (effects (font (size 1.27 1.27)) hide)
     )
@@
     (pin "1")
   )
-  (symbol (lib_id "Transistor_BJT:S8050") (at 129.54 118.11 0) (mirror y) (unit 1)
-    (in_bom yes) (on_board yes) (fields_autoplaced)
-    (property "Reference" "Q1" (id 0) (at 124.46 116.8399 0)
-      (effects (font (size 1.27 1.27)) (justify left))
-    )
-    (property "Value" "S8050" (id 1) (at 124.46 119.3799 0)
-      (effects (font (size 1.27 1.27)) (justify left))
-    )
-    (property "Footprint" "Package_TO_SOT_THT:TO-92_Inline" (id 2) (at 124.46 120.015 0)
+  (symbol (lib_name "S8050_1") (lib_id "Transistor_BJT:S8050") (at 129.54 118.11 0) (mirror y) (unit 1)
+    (in_bom yes) (on_board yes) (fields_autoplaced)
+    (property "Reference" "Q1" (id 0) (at 134.62 116.8399 0)
+      (effects (font (size 1.27 1.27)) (justify left))
+    )
+    (property "Value" "S8050" (id 1) (at 134.62 119.3799 0)
+      (effects (font (size 1.27 1.27)) (justify left))
+    )
+    (property "Footprint" "footprint-lib:S8050,J3Y,SOT23" (id 2) (at 134.62 120.015 0)
       (effects (font (size 1.27 1.27) italic) (justify left) hide)
     )
@@
       (effects (font (size 1.27 1.27)) (justify left) hide)
     )
-    (pin "1")
-    (pin "2")
-    (pin "3")
+    (pin "E")
+    (pin "B")
+    (pin "C")
   )
   (symbol (lib_id "taobao-r:R123,0805") (at 40.64 66.04 90) (unit 1)
@@
       (effects (font (size 1.27 1.27)) (justify left))
     )
-    (property "Footprint" "" (id 2) (at 257.81 116.84 90)
+    (property "Footprint" "Diode_SMD:D_SMA" (id 2) (at 257.81 116.84 90)
       (effects (font (size 1.27 1.27)) hide)
     )
@@
       (effects (font (size 1.27 1.27)) (justify left))
     )
-    (property "Footprint" "Capacitor_SMD:C_0805_2012Metric_Pad1.15x1.40mm_HandSolder" (id 2) (at 154.94 143.51 0)
+    (property "Footprint" "Capacitor_SMD:C_0805_2012Metric" (id 2) (at 154.94 143.51 0)
       (effects (font (size 1.27 1.27)) hide)
     )
@@
     (property "Reference" "R13" (id 0) (at 143.51 111.76 90))
     (property "Value" "R123,0805" (id 1) (at 143.51 114.3 90))
-    (property "Footprint" "Resistor_SMD:R_0805_2012Metric_Pad1.15x1.40mm_HandSolder" (id 2) (at 143.51 118.11 0)
+    (property "Footprint" "Resistor_SMD:R_0805_2012Metric" (id 2) (at 143.51 118.11 0)
       (effects (font (size 1.27 1.27)) hide)
     )
@@
       (effects (font (size 1.27 1.27)) (justify left))
     )
-    (property "Footprint" "Resistor_SMD:R_0805_2012Metric_Pad1.15x1.40mm_HandSolder" (id 2) (at 331.47 114.3 0)
+    (property "Footprint" "Resistor_SMD:R_0805_2012Metric" (id 2) (at 331.47 114.3 0)
       (effects (font (size 1.27 1.27)) hide)
     )
@@
     (property "Reference" "R12" (id 0) (at 204.47 138.43 90))
     (property "Value" "R471,0805" (id 1) (at 204.47 140.97 90))
-    (property "Footprint" "Resistor_SMD:R_0805_2012Metric_Pad1.15x1.40mm_HandSolder" (id 2) (at 204.47 134.62 0)
+    (property "Footprint" "Resistor_SMD:R_0805_2012Metric" (id 2) (at 204.47 134.62 0)
       (effects (font (size 1.27 1.27)) hide)
     )
@@
     (pin "1")
   )
-  (symbol (lib_id "Transistor_BJT:S8050") (at 129.54 138.43 180) (unit 1)
-    (in_bom yes) (on_board yes) (fields_autoplaced)
-    (property "Reference" "Q2" (id 0) (at 124.46 137.1599 0)
-      (effects (font (size 1.27 1.27)) (justify left))
-    )
-    (property "Value" "S8050" (id 1) (at 124.46 139.6999 0)
-      (effects (font (size 1.27 1.27)) (justify left))
-    )
-    (property "Footprint" "Package_TO_SOT_THT:TO-92_Inline" (id 2) (at 124.46 136.525 0)
-      (effects (font (size 1.27 1.27) italic) (justify left) hide)
-    )
-    (property "Datasheet" "http://www.unisonic.com.tw/datasheet/S8050.pdf" (id 3) (at 129.54 138.43 0)
-      (effects (font (size 1.27 1.27)) (justify left) hide)
-    )
-    (pin "1")
-    (pin "2")
-    (pin "3")
-  )
   (symbol (lib_id "taobao-c:C104,0805") (at 162.56 143.51 0) (unit 1)
     (in_bom yes) (on_board yes) (fields_autoplaced)
@@
       (effects (font (size 1.27 1.27)) (justify left))
     )
-    (property "Footprint" "Capacitor_SMD:C_0805_2012Metric_Pad1.15x1.40mm_HandSolder" (id 2) (at 162.56 143.51 0)
+    (property "Footprint" "Capacitor_SMD:C_0805_2012Metric" (id 2) (at 162.56 143.51 0)
       (effects (font (size 1.27 1.27)) hide)
     )
@@
       (effects (font (size 1.27 1.27)) (justify left))
     )
-    (property "Footprint" "Capacitor_SMD:C_0805_2012Metric_Pad1.15x1.40mm_HandSolder" (id 2) (at 44.45 191.77 0)
+    (property "Footprint" "Capacitor_SMD:C_0805_2012Metric" (id 2) (at 44.45 191.77 0)
       (effects (font (size 1.27 1.27)) hide)
     )
@@
       (effects (font (size 1.27 1.27)) (justify left))
     )
-    (property "Footprint" "Capacitor_SMD:C_0805_2012Metric_Pad1.15x1.40mm_HandSolder" (id 2) (at 49.53 129.54 0)
+    (property "Footprint" "Capacitor_SMD:C_0805_2012Metric" (id 2) (at 49.53 129.54 0)
       (effects (font (size 1.27 1.27)) hide)
     )
@@
     (property "Reference" "R14" (id 0) (at 143.51 132.08 90))
     (property "Value" "R123,0805" (id 1) (at 143.51 134.62 90))
-    (property "Footprint" "Resistor_SMD:R_0805_2012Metric_Pad1.15x1.40mm_HandSolder" (id 2) (at 143.51 138.43 0)
+    (property "Footprint" "Resistor_SMD:R_0805_2012Metric" (id 2) (at 143.51 138.43 0)
       (effects (font (size 1.27 1.27)) hide)
     )
@@
     (pin "1")
   )
+  (symbol (lib_name "S8050_1") (lib_id "Transistor_BJT:S8050") (at 129.54 138.43 180) (unit 1)
+    (in_bom yes) (on_board yes) (fields_autoplaced)
+    (property "Reference" "Q2" (id 0) (at 124.46 137.1599 0)
+      (effects (font (size 1.27 1.27)) (justify left))
+    )
+    (property "Value" "S8050" (id 1) (at 124.46 139.6999 0)
+      (effects (font (size 1.27 1.27)) (justify left))
+    )
+    (property "Footprint" "footprint-lib:S8050,J3Y,SOT23" (id 2) (at 134.62 136.525 0)
+      (effects (font (size 1.27 1.27) italic) (justify left) hide)
+    )
+    (property "Datasheet" "http://www.unisonic.com.tw/datasheet/S8050.pdf" (id 3) (at 129.54 138.43 0)
+      (effects (font (size 1.27 1.27)) (justify left) hide)
+    )
+    (pin "B")
+    (pin "C")
+    (pin "E")
+  )
   (symbol (lib_id "taobao-c:C471,0805") (at 76.2 194.31 0) (unit 1)
     (in_bom yes) (on_board yes) (fields_autoplaced)
@@
       (effects (font (size 1.27 1.27)) (justify left))
     )
-    (property "Footprint" "Capacitor_SMD:C_0805_2012Metric_Pad1.15x1.40mm_HandSolder" (id 2) (at 76.2 194.31 0)
+    (property "Footprint" "Capacitor_SMD:C_0805_2012Metric" (id 2) (at 76.2 194.31 0)
       (effects (font (size 1.27 1.27)) hide)
     )
@@
       (effects (font (size 1.27 1.27)) (justify left))
     )
-    (property "Footprint" "Capacitor_SMD:C_0805_2012Metric_Pad1.15x1.40mm_HandSolder" (id 2) (at 222.25 133.35 0)
-      (effects (font (size 1.27 1.27)) hide)
-    )
+    (property "Footprint" "Capacitor_SMD:C_0805_2012Metric" (id 2) (at 222.25 133.35 0)
+      (effects (font (size 1.27 1.27)) hide)
+    )

Commit message: update,
Parts:
- C1: renamed from C?; footprint Capacitor_SMD:CP_Elec_6.3x7.7 -> Capacitor_Tantalum_SMD:CP_EIA-3528-12_Kemet-T
- SW1, SW3: footprint footprint-lib:microswitch_6_6_5 -> footprint-lib:SW_SPST_CK_RS282G05A3
- U1: footprint footprint-lib:ESP-12E -> footprint-lib:ESP-12E_NO_HOLE
- U2: footprint Package_SO:SSOP-20_5.3x7.2mm_P0.65mm -> Package_SO:SOP-16_3.9x9.9mm_P1.27mm
- gave numbers to parts that had none: 1
Connections:
- no-connect marks 13 -> 12
