File: hardware/42-stepper-motor-driver-tryout.kicad_pcb (KiCad board)
At the start: 2 copper layers, 42 x 42 mm, 66 parts, among them J1 Conn_01x04, J2 Conn_01x04, J3 Conn_01x04, Q1 S8050, Q2 S8050, SW1 microswitch_6_6_5, SW3 microswitch_6_6_5, U1 ESP-12E, U2 CH340G, U3 USB_Micro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

Commit message: update,
Parts:
- C12, C13, C14, C15, C16, C3, C6, C7, C8, R10, R12, R16, R17, R18, R22, R3, R8: moved to F.Cu
- R19, R20: moved to B.Cu
- moved C6 12.3 mm to (27.5, 30.5), turned to -90 degrees
- moved C13 10.2 mm to (8.77, 21.5), turned to 0 degrees
- moved C8 9.96 mm to (30.5, 26.0), turned to 90 degrees
- moved JP2 9.09 mm to (31.0, 36.0)
- moved R17 8.82 mm to (8.75, 19.5), turned to 180 degrees
- moved R3 8.55 mm to (8.75, 15.5), turned to 0 degrees
- moved C3 8.21 mm to (8.77, 17.5), turned to 180 degrees
- moved C14 8.00 mm to (5.34, 22.0), turned to 180 degrees
- moved R11 7.74 mm to (26.8, 27.0)
- moved C10 7.34 mm to (16.5, 31.0)
- moved C7 7.02 mm to (32.5, 26.0), turned to 90 degrees
- moved R9 6.93 mm to (24.5, 27.0)
- moved R2 6.46 mm to (22.5, 27.0)
- moved C12 6.21 mm to (8.77, 23.8), turned to 0 degrees
- moved R4 6.01 mm to (20.5, 27.0)
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Other:
- outline, holes or cut-outs redrawn
- copper layers 2 -> 4
